File: T245Controller_rev1.brd (EAGLE design)
At the start: 160 x 100 mm, 72 parts, among them IC2 LM4041A12LP, IC4 LT1078, Q1 BSC040N08NS5ATMA1, Q2 BSC040N08NS5ATMA1, U1 ARDUINO_NANO_A000005, U2 MAX5035DUPA+, X1 MKDSN1,5/2-5,08, X3 MKDSN1,5/3-5,08

Commit message: Add files via upload
Parts:
- removed R1: (no value), rcl:0207/10
- removed R11: MSR1-0R01F1, rcl:0207/12
- removed X1: MKDSN1,5/2-5,08, con-phoenix-508:MKDSN1,5/2-5,08
- added 1K: (no value), rcl:0207/10
- added SHUNT: MSR1-0R01F1, rcl:0207/12
- added X2: MKDSN1,5/3-5,08, con-phoenix-508:MKDSN1,5/3-5,08
- Q1, Q2: device transistor-fet:TO220 -> transistor-power:TO220BV
- Q4, Q5: value (none) -> IRF540; device transistor-fet:TO220 -> transistor-power:TO220BV
- moved C14 261.9 mm to (51.8, 33.0), turned to 180 degrees
- moved D6 238.0 mm to (52.1, 61.0), turned to 90 degrees
- moved T2 237.5 mm to (83.5, 44.5), turned to 270 degrees
- moved D9 236.5 mm to (47.0, 61.0), turned to 270 degrees
- moved D12 234.2 mm to (22.9, 58.4)
- moved D10 234.1 mm to (40.6, 61.0), turned to 270 degrees
- moved D11 232.1 mm to (34.3, 61.0), turned to 90 degrees
- moved C13 230.0 mm to (12.7, 53.3)
- moved R28 227.8 mm to (20.8, 33.0), turned to 270 degrees
- moved X3 218.2 mm to (86.7, 10.2), turned to 180 degrees
- moved R29 217.2 mm to (11.4, 22.9), turned to 180 degrees
- moved D1 213.5 mm to (84.8, 58.4), turned to 180 degrees
- moved D4 211.7 mm to (84.8, 63.5), turned to 180 degrees
- moved C9 208.3 mm to (77.2, 31.8), turned to 270 degrees
- moved OC2 207.9 mm to (10.2, 35.6), turned to 270 degrees
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Connections:
- removed net N$14: F1.1, X1.1
- removed net V+: D2.A, D6.C, D9.A, F1.2, Q1.2, Q4.2, R15.1
- new net N$24: F1.1, X2.3
- net 24VAC: now also D2.A, D6.C, D9.A, F1.2, Q1.D, Q4.D, R15.1
- net C1: now also SHUNT.2; no longer R11.2
- net C2: now also Q2.D; no longer Q2.2
- net GNDA: now also Q5.D, SHUNT.1, X2.2; no longer Q5.2, R11.1, X1.2
- net N$2: now also 1K.1; no longer R1.1
- net N$20: now also Q4.S, Q5.S; no longer Q4.3, Q5.3
- net N$23: now also Q4.G, Q5.G; no longer Q4.1, Q5.1
- net N$3: now also Q1.G, Q2.G; no longer Q1.1, Q2.1
- net N$4: now also Q1.S, Q2.S; no longer Q1.3, Q2.3
- net OPTO: now also 1K.2; no longer R1.2
- net PE: now also X2.1
Routing:
- net 24VAC: track 0.00 -> 126.7 mm, vias 0 -> 1
- net N$4: track 0.00 -> 94.6 mm, vias 0 -> 2
- net 5VDC: track 0.00 -> 60.4 mm
- net 7VDC: track 31.0 -> 89.8 mm, vias 0 -> 1
- net N$21: track 0.00 -> 57.6 mm
- net OPTO: track 0.00 -> 56.5 mm, vias 0 -> 2
- net VREF: track 0.00 -> 54.5 mm
- net THERM: track 0.00 -> 54.0 mm
- net N$29: track 0.00 -> 50.4 mm
- net N$3: track 0.00 -> 47.5 mm
- net TCOP: track 0.00 -> 47.3 mm
- net C3: track 0.00 -> 44.9 mm
- net N$13: track 0.00 -> 41.5 mm
- net SHUNTOP: track 0.00 -> 39.1 mm
- net N$30: track 0.00 -> 36.8 mm
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- added copper zone on layer 1, net 24VAC
- added copper zone on layer 1, net C1
- added copper zone on layer 1, net C2
- added copper zone on layer 1, net N$24
- added copper zone on layer 1, net N$4
Other:
- board size 160 x 100 mm -> 100 x 100 mm

Commit message: Add files via upload
Parts:
- removed 1K: (no value), rcl:0207/10
- removed IC4: LT1078, analog-devices:DIL08
- removed R10: 10k, rcl:0207/10
- removed R28: 100k, rcl:0207/10
- removed R29: 1M, rcl:0207/10
- removed R8: 22k, rcl:0207/10
- removed R9: 47k, rcl:0207/10
- removed T1, T3: (no value), transistor-neu-to92:TO92-EBC
- added NTC: Thermistor 100k, rcl:0207/10
- added R1: 1M, rcl:0207/10
- added R11: 1k, rcl:0207/10
- added TVS1, TVS2: P6KE51CA, P6KE51CA:P6KESERIES_LTF
- added U3: LT1078, analog-devices:DIL08
- C13: value 1n -> 100n
- C14, C2: value 100n -> 10u
- C3: value 10u -> 100n; device rcl:E2,5-6 -> rcl:C050-024X044
- C5: value 10u -> ESC686M035AE3AA; device rcl:C050-024X044 -> rcl:E2,5-6
- C6: value ESC686M035AE3AA -> 100n; device rcl:E2,5-6 -> rcl:C050-024X044
- C8: value 100n -> 10u; device rcl:C050-024X044 -> rcl:E2,5-6
- D1: value 1N5245 -> (none); device diode:DO41Z10 -> diode:F126Z12
- D10, D9: value (none) -> 1N5245; device diode:F126Z12 -> diode:DO41Z10
- D11, D12: value (none) -> 1N3595; device diode:F126Z12 -> diode:D-7.5
- D3, D6, D7: device diode:F126Z12 -> diode:D-7.5
- D4: value 1N5245 -> (none); device diode:DO41Z10 -> diode:D-7.5
- D5, D8: value BZX55C39 -> (none); device diode:DO41Z10 -> diode:D-7.5
- Q4, Q5: value IRF540 -> (none); device transistor-power:TO220BV -> transistor-neu-to92:TO92-EBC
- R12: value 1k -> 470k
- R13: value 4.7k -> 47k
- R14: value 100k -> 22k
- R15: value 220 -> 4.7k
- R16: value 220 -> 250k
- R17: value Thermistor 100k -> 1k
- R18: value 100k -> 4.7k
- R19: value 1k -> 47k
- R20: value 4.7k -> 1k
- R21: value 1k -> 100k
- R22: value 47k -> 100k
- R24: value 100k -> 10k
- R25: value 100k -> 100
- R26: value 10k -> 1M
- R27: value 100 -> 100k
- R3: value 250k -> 10k
- R6: value 1M -> 1k
- R7: value 470k -> 100k
- moved R6 87.6 mm to (6.35, 12.7), turned to 90 degrees
- moved C6 86.4 mm to (11.4, 10.2), turned to 270 degrees
- moved R3 75.8 mm to (8.58, 82.5), turned to 180 degrees
- moved C8 72.0 mm to (67.0, 55.9), turned to 0 degrees
- moved R22 68.4 mm to (10.2, 64.8)
- moved Q4 66.3 mm to (19.1, 45.7), turned to 90 degrees
- moved Q5 66.2 mm to (14.0, 45.7), turned to 270 degrees
- moved R15 65.2 mm to (67.0, 24.1)
- moved R2 64.8 mm to (8.58, 77.5), turned to 0 degrees
- moved R16 60.2 mm to (67.0, 34.3), turned to 0 degrees
- moved C3 54.4 mm to (25.1, 90.6)
- moved R21 54.0 mm to (24.1, 53.3), turned to 0 degrees
- moved R17 48.5 mm to (67.0, 29.2), turned to 180 degrees
- moved R19 46.7 mm to (53.0, 11.4)
- moved D4 44.1 mm to (40.6, 63.5), turned to 270 degrees
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- renumbered IC2 to U4, T2 to Q3
Connections:
- removed net N$15: C10.1, IC4.5, R13.1
- removed net N$19: D8.C, R15.2
- removed net N$20: Q4.S, Q5.S, R14.1
- removed net N$23: D5.A, D8.A, Q4.G, Q5.G, R14.2
- net 24VAC: now also D1.A, D3.C, D4.A, D8.A, TVS2.1; no longer D2.A, D6.C, D7.A, D9.A, Q4.D, R15.1
- net 5VDC: now also C13.1, R27.1, U3.8; no longer C14.1, IC4.8, R28.1
- net 7VDC: now also C5.+; no longer C6.+
- net C1: now also R18.2, TVS1.1; no longer R20.2
- net C2: now also TVS1.2
- net C3: now also R15.2; no longer R13.2
- net GNDA: now also C13.2, C2.1, C5.-, C6.1, D11.A, D12.C, D2.A, D5.C, D6.A, R1.2, R17.2, R20.2, R26.1, R3.1, R7.1, TVS2.2, U3.4; no longer C14.2, C5.1, C6.-, C8.1, D10.A, D11.C, D3.A, IC4.4, Q5.D, R10.1, R12.2, R16.2, R18.1, R21.2, R29.1, R6.2
- net N$1: now also R16.2, R17.1, U3.6; no longer IC4.6, R12.1, R3.2
- net N$10: now also C2.2, D1.C, R2.2; no longer C5.2, D7.C, R9.2
- net N$11: now also C10.1, D11.C, D12.A, R15.1, U3.5; no longer D5.C, R16.1
- net N$12: now also C3.1; no longer C2.1
- net N$13: now also R13.1; no longer R2.1
- net N$16: now also D10.C, D9.C; no longer D1.C, D4.C
- net N$17: now also R2.1, R3.2; no longer R10.2, R9.1
- net N$2: now also R11.1; no longer 1K.1
- net N$21: now also C14.2, D3.A, D5.A, R25.1; no longer C13.2, D11.A, D6.A, R27.1
- net N$22: now also R26.2; no longer R29.2
- net N$25: now also R18.1, U3.3; no longer IC4.3, R20.1
- net N$26: now also D4.C, D6.C, D7.A, R21.2; no longer D10.C, D12.A, D9.C, R24.2
- net N$27: now also R19.2, R20.1, U3.2; no longer IC4.2, R21.1, R22.2
- net N$28: now also Q4.B, R21.1; no longer R24.1, T1.B
- net N$29: now also C14.1, D7.C, R22.1, R24.1; no longer C13.1, D12.C, R25.1, R26.1
- net N$3: now also D9.A, R14.1; no longer D1.A, R8.1
- net N$30: now also Q4.C, R22.2; no longer R25.2, T1.C
- net N$31: now also Q4.E, Q5.E, R25.2; no longer R27.2, T1.E, T3.E
- net N$32: now also R24.2; no longer R26.2
- net N$33: now also Q5.C; no longer T3.C
- net N$4: now also C8.-, D10.A, R12.1; no longer C3.-, D4.A, R7.1
- net N$5: now also R12.2; no longer R7.2
- net N$6: now also Q5.B; no longer T3.B
- net N$8: now also C3.2, D2.C; no longer C2.2, D3.C
- net N$9: now also C8.+, D8.C, R13.2, R14.2; no longer C3.+, D2.C, R2.2, R8.2
- net OPTO: now also R11.2; no longer 1K.2
- net PE: now also R1.1; no longer R6.1
- net SHUNTOP: now also R19.1, U3.1; no longer IC4.1, R22.1
- net TCOP: now also R16.1, U3.7; no longer IC4.7, R3.1
- net THERM: now also NTC.1, R7.2; no longer R17.1, R18.2
- net VREF: now also C6.2, NTC.2, R6.1; no longer C8.2, R17.2, R19.1
- net VREFPWR: now also R6.2; no longer R19.2
- net ZCINT: now also R27.2; no longer R28.2
Routing:
- net 24VAC: track 126.7 -> 68.4 mm, vias 1 -> 0
- net N$23: track 34.2 -> 0.00 mm
- net N$4: track 94.6 -> 76.1 mm, vias 2 -> 0
- net PE: track 27.5 -> 9.20 mm
- net N$20: track 15.7 -> 0.00 mm
- net OPTO: track 56.5 -> 41.3 mm, vias 2 -> 0
- net N$15: track 13.5 -> 0.00 mm
- net 5VDC: track 60.4 -> 71.8 mm
- net N$27: track 32.2 -> 42.7 mm
- net N$10: track 28.6 -> 38.7 mm
- net N$11: track 12.1 -> 21.9 mm
- net N$25: track 24.5 -> 34.2 mm
- net N$2: track 17.3 -> 9.23 mm
- net SHUNTOP: track 39.1 -> 46.6 mm
- net C3: track 44.9 -> 37.6 mm
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Other:
- outline, holes or cut-outs redrawn
