File: T245Controller_rev1.sch (EAGLE design)
At the start: 72 parts, among them IC2 LM4041A12LP, IC4 LT1078, Q1 BSC040N08NS5ATMA1, Q2 BSC040N08NS5ATMA1, Q4 IRF540, Q5 IRF540, U1 ARDUINO_NANO_A000005, U2 MAX5035DUPA+, X1 MKDSN1,5/2-5,08, X3 MKDSN1,5/3-5,08

Commit message: Add files via upload
Parts:
- removed X1: MKDSN1,5/2-5,08, con-phoenix-508:MKDSN1,5/2-5,08
- added X2: MKDSN1,5/3-5,08, con-phoenix-508:MKDSN1,5/3-5,08
- Q1, Q2, Q4, Q5: device transistor-fet:IRF540 -> transistor-power:IRF540
- renumbered R1 to 1K, R11 to SHUNT
Connections:
- removed net N$14: F1.1, X1-1.KL
- removed net V+: D2.A, D6.C, D9.A, F1.2, Q1.D, Q4.D, R15.1
- new net N$24: F1.1, X2-3.KL
- net 24VAC: now also D2.A, D6.C, D9.A, F1.2, Q1.D, Q4.D, R15.1
- net GNDA: now also X2-2.KL; no longer X1-2.KL
- net PE: now also X2-1.KL

Commit message: Add files via upload
Parts:
- removed R10: 10k, rcl:R-EU_0207/10
- removed R28: 100k, rcl:R-EU_0207/10
- removed R29: 1M, rcl:R-EU_0207/10
- removed R8: 22k, rcl:R-EU_0207/10
- removed R9: 47k, rcl:R-EU_0207/10
- removed T1, T3: (no value), transistor-neu-to92:2N5550-NPN-TO92-EBC
- added NTC: Thermistor 100k, rcl:R-EU_0207/10
- added R1: 1M, rcl:R-EU_0207/10
- added TVS1, TVS2: P6KE51CA, P6KE51CA:P6KE51CA
- C13: value 1n -> 100n
- C14, C2: value 100n -> 10u
- C3: value 10u -> 100n; device rcl:CPOL-EUE2.5-6 -> rcl:C-EU050-024X044
- C5: value 10u -> ESC686M035AE3AA; device rcl:C-EU050-024X044 -> rcl:CPOL-EUE2.5-6
- C6: value ESC686M035AE3AA -> 100n; device rcl:CPOL-EUE2.5-6 -> rcl:C-EU050-024X044
- C8: value 100n -> 10u; device rcl:C-EU050-024X044 -> rcl:CPOL-EUE2.5-6
- D1: value 1N5245 -> (none); device diode:ZENER-DIODEDO41Z10 -> diode:SCHOTTKY-DIODEF126Z12
- D10, D9: value (none) -> 1N5245; device diode:SCHOTTKY-DIODEF126Z12 -> diode:ZENER-DIODEDO41Z10
- D11, D12: value (none) -> 1N3595; device diode:SCHOTTKY-DIODEF126Z12 -> diode:DIODE-D-7.5
- D3, D6, D7: device diode:SCHOTTKY-DIODEF126Z12 -> diode:DIODE-D-7.5
- D4: value 1N5245 -> (none); device diode:ZENER-DIODEDO41Z10 -> diode:DIODE-D-7.5
- D5, D8: value BZX55C39 -> (none); device diode:ZENER-DIODEDO41Z10 -> diode:DIODE-D-7.5
- Q4, Q5: value IRF540 -> (none); device transistor-power:IRF540 -> transistor-neu-to92:2N5550-NPN-TO92-EBC
- R11: value (none) -> 1k
- R12: value 1k -> 470k
- R13: value 4.7k -> 47k
- R14: value 100k -> 22k
- R15: value 220 -> 4.7k
- R16: value 220 -> 250k
- R17: value Thermistor 100k -> 1k
- R18: value 100k -> 4.7k
- R19: value 1k -> 47k
- R20: value 4.7k -> 1k
- R21: value 1k -> 100k
- R22: value 47k -> 100k
- R24: value 100k -> 10k
- R25: value 100k -> 100
- R26: value 10k -> 1M
- R27: value 100 -> 100k
- R3: value 250k -> 10k
- R6: value 1M -> 1k
- R7: value 470k -> 100k
- renumbered 1K to R11, IC2 to U4, IC4 to U3, T2 to Q3
Connections:
- removed net N$15: C10.1, R13.1, U3B.IN+
- removed net N$19: D8.C, R15.2
- removed net N$20: Q4.S, Q5.S, R14.1
- removed net N$23: D5.A, D8.A, Q4.G, Q5.G, R14.2
- net 24VAC: now also D1.A, D3.C, D4.A, D8.A, TVS2.11; no longer D2.A, D6.C, D7.A, D9.A, Q4.D, R15.1
- net 5VDC: now also C13.1, R27.1; no longer C14.1, R28.1
- net 7VDC: now also C5.+; no longer C6.+
- net C1: now also R18.2, TVS1.11; no longer R20.2
- net C2: now also TVS1.12
- net C3: now also R15.2; no longer R13.2
- net GNDA: now also C13.2, C2.1, C5.-, C6.1, D11.A, D12.C, D2.A, D5.C, D6.A, R1.2, R17.2, R20.2, R26.1, R3.1, R7.1, TVS2.12; no longer C14.2, C5.1, C6.-, C8.1, D10.A, D11.C, D3.A, Q5.D, R10.1, R12.2, R16.2, R18.1, R21.2, R29.1, R6.2
- net N$1: now also R16.2, R17.1; no longer R12.1, R3.2
- net N$10: now also C2.2, D1.C, R2.2; no longer C5.2, D7.C, R9.2
- net N$11: now also C10.1, D11.C, D12.A, R15.1, U3B.IN+; no longer D5.C, R16.1
- net N$12: now also C3.1; no longer C2.1
- net N$13: now also R13.1; no longer R2.1
- net N$16: now also D10.C, D9.C; no longer D1.C, D4.C
- net N$17: now also R2.1, R3.2; no longer R10.2, R9.1
- net N$21: now also C14.2, D3.A, D5.A, R25.1; no longer C13.2, D11.A, D6.A, R27.1
- net N$22: now also R26.2; no longer R29.2
- net N$25: now also R18.1; no longer R20.1
- net N$26: now also D4.C, D6.C, D7.A, R21.2; no longer D10.C, D12.A, D9.C, R24.2
- net N$27: now also R19.2, R20.1; no longer R21.1, R22.2
- net N$28: now also Q4.B, R21.1; no longer R24.1, T1.B
- net N$29: now also C14.1, D7.C, R22.1, R24.1; no longer C13.1, D12.C, R25.1, R26.1
- net N$3: now also D9.A, R14.1; no longer D1.A, R8.1
- net N$30: now also Q4.C, R22.2; no longer R25.2, T1.C
- net N$31: now also Q4.E, Q5.E, R25.2; no longer R27.2, T1.E, T3.E
- net N$32: now also R24.2; no longer R26.2
- net N$33: now also Q5.C; no longer T3.C
- net N$4: now also C8.-, D10.A, R12.1; no longer C3.-, D4.A, R7.1
- net N$5: now also R12.2; no longer R7.2
- net N$6: now also Q5.B; no longer T3.B
- net N$8: now also C3.2, D2.C; no longer C2.2, D3.C
- net N$9: now also C8.+, D8.C, R13.2, R14.2; no longer C3.+, D2.C, R2.2, R8.2
- net PE: now also R1.1; no longer R6.1
- net SHUNTOP: now also R19.1; no longer R22.1
- net TCOP: now also R16.1; no longer R3.1
- net THERM: now also NTC.1, R7.2; no longer R17.1, R18.2
- net VREF: now also C6.2, NTC.2, R6.1; no longer C8.2, R17.2, R19.1
- net VREFPWR: now also R6.2; no longer R19.2
- net ZCINT: now also R27.2; no longer R28.2
Other:
- note added: "P6KE51CA TVS Diode"
- note added: "Use low Vf Schottkys"
- note removed: "Use low Cgate MOSFETs"
- moved on the sheet: C10, C12, C13, C14, C2, D2, R12, R13, R14, R15, R16, R17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
