File: T245Controller_rev0.brd (EAGLE design)
At the start: 100 x 100 mm, 71 parts, among them Q1 BSC040N08NS5ATMA1, Q2 BSC040N08NS5ATMA1, U1 ARDUINO_NANO_A000005, U2 MAX5035DUPA+, U3 LT1078, U4 LM4041A12LP, X2 MKDSN1,5/3-5,08, X3 MKDSN1,5/3-5,08

Commit message: Add files via upload
Parts:
- moved C5 1.27 mm to (34.9, 95.8)
- moved L1 1.27 mm to (40.3, 86.4)
- moved D2 1.03 mm to (30.5, 87.6)
Routing:
- net N$8: track 26.4 -> 27.1 mm
- net 7VDC: track 83.5 -> 83.0 mm
Changed lines of the file:
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@@
 <wire x1="3" y1="0" x2="97" y2="0" width="0" layer="20"/>
 <wire x1="100" y1="3" x2="100" y2="97" width="0" layer="20"/>
-<circle x="39.06" y="86.36" radius="7.493" width="0.1524" layer="21"/>
+<circle x="40.33" y="86.36" radius="7.493" width="0.1524" layer="21"/>
 <hole x="3" y="97" drill="3.2"/>
 <hole x="3" y="3" drill="3.2"/>
@@
 <attribute name="SPICEPREFIX" value="C" x="25.09" y="93.091" size="1.778" layer="27" display="off"/>
 </element>
-<element name="D2" library="diode" library_urn="urn:adsk.eagle:library:210" package="F126Z12" package3d_urn="urn:adsk.eagle:package:43358/1" value="" x="29.789" y="86.868" smashed="yes" rot="R90">
-<attribute name="NAME" x="33.091" y="85.979" size="1.27" layer="25" ratio="10" rot="R90"/>
-<attribute name="POPULARITY" value="1" x="29.789" y="86.868" size="1.778" layer="27" rot="R90" display="off"/>
-<attribute name="VALUE" x="32.456" y="84.582" size="1.27" layer="27" ratio="10" rot="R90"/>
-</element>
-<element name="L1" library="rcl" library_urn="urn:adsk.eagle:library:334" package="0207/10" package3d_urn="urn:adsk.eagle:package:23491/2" value="SBC7-221-132" x="39.06" y="86.36" smashed="yes" rot="R90">
-<attribute name="NAME" x="41.727" y="85.344" size="1.27" layer="25" ratio="10" rot="R90"/>
-<attribute name="POPULARITY" value="2" x="39.06" y="86.36" size="1.778" layer="27" rot="R90" display="off"/>
-<attribute name="SPICEPREFIX" value="L" x="39.06" y="86.36" size="1.778" layer="27" rot="R90" display="off"/>
+<element name="D2" library="diode" library_urn="urn:adsk.eagle:library:210" package="F126Z12" package3d_urn="urn:adsk.eagle:package:43358/1" value="" x="30.48" y="87.63" smashed="yes" rot="R90">
+<attribute name="NAME" x="33.782" y="86.741" size="1.27" layer="25" ratio="10" rot="R90"/>
+<attribute name="POPULARITY" value="1" x="30.48" y="87.63" size="1.778" layer="27" rot="R90" display="off"/>
+<attribute name="VALUE" x="33.147" y="85.344" size="1.27" layer="27" ratio="10" rot="R90"/>
+</element>
+<element name="L1" library="rcl" library_urn="urn:adsk.eagle:library:334" package="0207/10" package3d_urn="urn:adsk.eagle:package:23491/2" value="SBC7-221-132" x="40.33" y="86.36" smashed="yes" rot="R90">
+<attribute name="NAME" x="42.997" y="85.344" size="1.27" layer="25" ratio="10" rot="R90"/>
+<attribute name="POPULARITY" value="2" x="40.33" y="86.36" size="1.778" layer="27" rot="R90" display="off"/>
+<attribute name="SPICEPREFIX" value="L" x="40.33" y="86.36" size="1.778" layer="27" rot="R90" display="off"/>
 </element>
 <element name="C4" library="rcl" library_urn="urn:adsk.eagle:library:334" package="C050-024X044" package3d_urn="urn:adsk.eagle:package:23643/1" value="100n" x="17.4864" y="94.908596875" smashed="yes" rot="R315">
@@
 <attribute name="SPICEPREFIX" value="C" x="21.28" y="80.01" size="1.778" layer="27" display="off"/>
 </element>
-<element name="C5" library="rcl" library_urn="urn:adsk.eagle:library:334" package="E2,5-6" package3d_urn="urn:adsk.eagle:package:23349/1" value="ESC686M035AE3AA" x="33.599" y="95.758" smashed="yes" rot="R225">
-<attribute name="NAME" x="31.012775" y="99.652515625" size="1.27" layer="25" ratio="10" rot="R225"/>
-<attribute name="POPULARITY" value="26" x="33.599" y="95.758" size="1.778" layer="27" rot="R225" display="off"/>
-<attribute name="SPICEPREFIX" value="C" x="33.599" y="95.758" size="1.778" layer="27" rot="R225" display="off"/>
+<element name="C5" library="rcl" library_urn="urn:adsk.eagle:library:334" package="E2,5-6" package3d_urn="urn:adsk.eagle:package:23349/1" value="ESC686M035AE3AA" x="34.869" y="95.758" smashed="yes" rot="R225">
+<attribute name="NAME" x="31.266775" y="98.636515625" size="1.27" layer="25" ratio="10" rot="R225"/>
+<attribute name="POPULARITY" value="26" x="34.869" y="95.758" size="1.778" layer="27" rot="R225" display="off"/>
+<attribute name="SPICEPREFIX" value="C" x="34.869" y="95.758" size="1.778" layer="27" rot="R225" display="off"/>
 </element>
 <element name="F1" library="fuse" library_urn="urn:adsk.eagle:library:233" package="SH22,5A" package3d_urn="urn:adsk.eagle:package:14070/1" value="" x="86.05" y="82.55" smashed="yes" rot="R270">
@@
 <contactref element="R4" pad="2"/>
 <contactref element="C5" pad="+"/>
-<wire x1="39.06" y1="91.44" x2="39.06" y2="91.519075" width="2.54" layer="1"/>
-<wire x1="39.06" y1="91.519075" x2="34.497025" y2="96.656025" width="2.54" layer="1"/>
-<wire x1="39.06" y1="91.44" x2="48.133" y2="82.367" width="1.016" layer="1"/>
-<wire x1="34.497025" y1="96.656025" x2="34.361" y2="96.52" width="0.508" layer="1"/>
+<wire x1="40.33" y1="91.44" x2="40.33" y2="91.519075" width="2.54" layer="1"/>
+<wire x1="40.33" y1="91.519075" x2="35.767025" y2="96.656025" width="2.54" layer="1"/>
+<wire x1="40.33" y1="91.44" x2="48.133" y2="83.637" width="1.016" layer="1"/>
+<wire x1="35.767025" y1="96.656025" x2="35.631" y2="96.52" width="0.508" layer="1"/>
 <wire x1="13.66" y1="87.63" x2="16.002" y2="89.972" width="0.6096" layer="1"/>
 <wire x1="16.002" y1="89.972" x2="16.002" y2="93.091" width="0.6096" layer="1"/>
@@
 <wire x1="42.8832" y1="48.4505" x2="42.1005" y2="48.4505" width="1.016" layer="1"/>
 <wire x1="42.1005" y1="48.4505" x2="41.91" y2="48.26" width="1.016" layer="1"/>
-<wire x1="48.133" y1="82.367" x2="48.133" y2="60.833" width="1.016" layer="1"/>
+<wire x1="48.133" y1="83.637" x2="48.133" y2="60.833" width="1.016" layer="1"/>
 <wire x1="48.133" y1="60.833" x2="44.45" y2="57.15" width="1.016" layer="1"/>
 <wire x1="44.45" y1="57.15" x2="44.45" y2="50.0173" width="1.016" layer="1"/>
 <wire x1="44.45" y1="50.0173" x2="42.8832" y2="48.4505" width="1.016" layer="1"/>
-<wire x1="34.497025" y1="96.656025" x2="34.417" y2="96.901" width="0" layer="19" extent="1-1"/>
+<wire x1="35.631" y1="96.52" x2="34.417" y2="96.901" width="0" layer="19" extent="1-1"/>
 </signal>
 <signal name="N$10">
@@
 <contactref element="D2" pad="C"/>
 <contactref element="L1" pad="1"/>
-<wire x1="39.06" y1="81.28" x2="37.028" y2="83.312" width="2.54" layer="1"/>
-<wire x1="37.028" y1="83.312" x2="32.583" y2="83.312" width="2.54" layer="1"/>
-<wire x1="32.583" y1="83.312" x2="29.789" y2="80.518" width="2.54" layer="1"/>
+<wire x1="40.33" y1="81.28" x2="38.298" y2="83.312" width="2.54" layer="1"/>
+<wire x1="38.298" y1="83.312" x2="32.512" y2="83.312" width="2.54" layer="1"/>
+<wire x1="32.512" y1="83.312" x2="30.48" y2="81.28" width="2.54" layer="1"/>
 <wire x1="28.138" y1="81.915" x2="28.138" y2="92.583" width="0.6096" layer="1"/>
 <wire x1="27.63" y1="93.091" x2="28.138" y2="92.583" width="0.6096" layer="1"/>
-<wire x1="29.789" y1="80.518" x2="27.757" y2="82.55" width="2.54" layer="1"/>
-<wire x1="27.757" y1="82.55" x2="26.868" y2="82.55" width="2.54" layer="1"/>
+<wire x1="30.48" y1="81.28" x2="29.21" y2="82.55" width="2.54" layer="1"/>
+<wire x1="29.21" y1="82.55" x2="26.868" y2="82.55" width="2.54" layer="1"/>
 <wire x1="26.868" y1="82.55" x2="28.138" y2="81.915" width="0" layer="19" extent="1-1"/>
 <wire x1="26.36" y1="82.55" x2="26.868" y2="82.55" width="0" layer="19" extent="1-1"/>
